Commit message: fixed odometry and added move_base

File: multi_jackal_description/urdf/accessories.urdf.xacro (robot description, xacro)
@@ -9,4 +9,5 @@
     jackal_base/launch/base.launch
   -->
+  <xacro:arg name="namespace"                      default="jackal0" />
   <!-- Macros to generate standoffs for offset payload mounting. -->
   <xacro:include filename="accessories/standoffs.urdf.xacro" />

File: multi_jackal_description/urdf/accessories/sick_lms1xx_mount.urdf.xacro (robot description, xacro)
@@ -26,7 +26,8 @@
 -->
 <robot xmlns:xacro="http://www.ros.org/wiki/xacro">
+  <xacro:arg name="namespace"                      default="jackal0" />
   <xacro:include filename="$(find lms1xx)/urdf/sick_lms1xx.urdf.xacro" />
   <xacro:macro name="sick_lms1xx_mount" params="prefix topic">
-    <sick_lms1xx frame="${prefix}_laser" topic="${topic}" robot_namespace="$(arg namespace)" />
+    <sick_lms1xx frame="${prefix}_laser_pp" topic="${topic}" robot_namespace="$(arg namespace)" />
     <link name="${prefix}_laser_mount">
       <visual>
@@ -43,5 +44,5 @@
       <origin xyz="0 0 0.149" rpy="0 0 0" />
       <parent link="${prefix}_laser_mount" />
-      <child link="${prefix}_laser" />
+      <child link="${prefix}_laser_pp" />
     </joint>
     <gazebo reference="${prefix}_laser_mount">

File: multi_jackal_description/urdf/jackal.urdf.xacro (robot description, xacro)
@@ -4,4 +4,5 @@
      Requires the arguments: $namespace, $id -->
 <robot name="jackal" xmlns:xacro="http://www.ros.org/wiki/xacro">
+  <xacro:arg name="namespace"                      default="jackal0" />
   <xacro:property name="PI"                        value="3.1415926535897931" />
   <xacro:property name="wheelbase"                 value="0.262" />
